Commit message: add gps urdf

File: iqr_jh_description/urdf/iqr_jh_robot.urdf.xacro (robot description, xacro)
@@ -7,4 +7,5 @@
   <xacro:include filename="$(find ${package_name})/urdf/zed2.xacro"/>
   <xacro:include filename="$(find ${package_name})/urdf/vlp16.xacro"/>
+  <xacro:include filename="$(find ${package_name})/urdf/gps_antenna.xacro"/>
   <xacro:include filename="$(find ${package_name})/urdf/livox_horizon.xacro"/>
   <xacro:include filename="$(find ${package_name})/urdf/sensor_support.xacro"/>
@@ -30,3 +31,7 @@
     <origin xyz="0 0 0" rpy="0 0 0"/>
   </xacro:sensor_d435>
+  <!-- GPS -->
+  <xacro:gps_antenna package="${package_name}" name="rtk" parent="rtk_gps_mount_link">
+    <origin xyz="0 0 0.02" rpy="0 0 0"/>
+  </xacro:gps_antenna>
 </robot>
